File: Hardware/SparkFun_LIS3DH.kicad_sch (KiCad schematic)
At the start: 29 parts, among them J1 Conn_01x02, J2 Conn_01x05, J3 Qwiic_RA, J4 I2C, J5 Qwiic_RA, U1 LIS3DH

Commit message: Updates LIS3DH according to new changes
Parts:
- U1: footprint SparkFun-Sensor:LGA-16-3X3 -> SparkFun-Sensor:ST_LGA-16_3x3mm_P0.5mm_5x3
Changed lines of the file:
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@@
 			)
 		)
-		(property "Footprint" "SparkFun-Sensor:LGA-16-3X3"
+		(property "Footprint" "SparkFun-Sensor:ST_LGA-16_3x3mm_P0.5mm_5x3"
 			(at 80.518 99.822 0)
 			(effects

Commit message: Moves v10 in board, updates IC symbol, and fixes various text
Other:
- title: SparkFun Ambient Light Sensor - VEML7700 -> SparkFun Triple Axis Accelerometer - LIS3DH (Qwiic)
Changed lines of the file:
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@@
 	(paper "USLetter")
 	(title_block
-		(title "SparkFun Ambient Light Sensor - VEML7700")
+		(title "SparkFun Triple Axis Accelerometer - LIS3DH (Qwiic)")
 		(date "2025-04-24")
 		(rev "v10")
 		(company "SparkFun Electronics")
-		(comment 1 "Original Design by: Paul Clark")
-		(comment 2 "Designed by: Elias Santistevan")
+		(comment 1 "Designed by: Elias Santistevan")
 	)
 	(text "Triple Axis Accelerometer - LIS3DH"
@@
 	)
 	(junction
-		(at 67.31 81.28)
-		(diameter 0)
-		(color 0 0 0 0)
-	)
-	(junction
 		(at 134.62 66.04)
 		(diameter 0)
@@
 	(wire
 		(pts
-			(xy 68.58 81.28) (xy 67.31 81.28)
-		)
-		(stroke
-			(width 0)
-			(type default)
-		)
-	)
-	(wire
-		(pts
 			(xy 53.34 137.16) (xy 52.07 137.16)
 		)
@@
 	(wire
 		(pts
-			(xy 67.31 81.28) (xy 67.31 83.82)
-		)
-		(stroke
-			(width 0)
-			(type default)
-		)
-	)
-	(wire
-		(pts
 			(xy 52.07 58.42) (xy 55.88 58.42)
 		)
@@
 	(wire
 		(pts
-			(xy 67.31 69.85) (xy 67.31 81.28)
+			(xy 67.31 69.85) (xy 67.31 83.82)
 		)
 		(stroke
@@
 				)
 				(justify left bottom)
-				(hide yes)
 			)
 		)
@@
 				)
 				(justify left top)
-				(hide yes)
 			)
 		)
