File: Hardware/Micro/SparkFun_LIS3DH_Micro.kicad_sch (KiCad schematic)
At the start: 27 parts, among them J1 PTH_1x1mm, J2 Qwiic_RA, J5 PTH_1x1mm, U1 LIS3DH

Commit message: Fixes design information in title bar
Other:
- title: SparkFun Ambient Light Sensor - VEML7700 -> SparkFun Triple Axis Accelerometer - LIS3DH
Changed lines of the file:
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@@
 	(paper "USLetter")
 	(title_block
-		(title "SparkFun Ambient Light Sensor - VEML7700")
+		(title "SparkFun Triple Axis Accelerometer - LIS3DH")
 		(date "2025-04-24")
 		(rev "v10")
 		(company "SparkFun Electronics")
-		(comment 1 "Original Design by: Paul Clark")
-		(comment 2 "Designed by: Elias Santistevan")
+		(comment 1 "Designed by: Elias Santistevan")
 	)
 	(text "Testpoints"

Commit message: Fixes silk on micro, and adds note about 22AWG wire with PTH
Other:
- note added: "Plated through holes can fit 22AWG wire or smaller."
Changed lines of the file:
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@@
 		(comment 1 "Designed by: Elias Santistevan")
+	)
+	(text "Plated through holes can fit\n22AWG wire or smaller."
+		(exclude_from_sim no)
+		(at 107.442 127.762 0)
+		(effects
+			(font
+				(size 1.27 1.27)
+				(thickness 0.1588)
+			)
+		)
 	)
 	(text "Testpoints"

Commit message: Updates LIS3DH in the micro board according to new changes
Parts:
- U1: footprint SparkFun-Sensor:LGA-16-3X3 -> SparkFun-Sensor:ST_LGA-16_3x3mm_P0.5mm_5x3
Changed lines of the file:
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@@
 			)
 		)
-		(property "Footprint" "SparkFun-Sensor:LGA-16-3X3"
+		(property "Footprint" "SparkFun-Sensor:ST_LGA-16_3x3mm_P0.5mm_5x3"
 			(at 80.518 99.822 0)
 			(effects

Commit message: Updates the 1 mm PTH part
Parts:
- D1: footprint SparkFun-LED:LED_0402_1005Metric -> SparkFun-LED:LED_0402_1005Metric_Red; PROD_ID DIO-25000 -> DIO-16757
- J1, J5: footprint SparkFun-Connector:1x01_PTH_1x1mm -> SparkFun-Connector:1x01_1x1mm
Changed lines of the file:
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@@
 			)
 		)
-		(property "Footprint" "SparkFun-Connector:1x01_PTH_1x1mm"
+		(property "Footprint" "SparkFun-Connector:1x01_1x1mm"
 			(at 106.68 147.32 0)
 			(effects
@@
 	)
 	(symbol
+		(lib_name "Conn_01x01_PTH_1x1mm_1")
 		(lib_id "SparkFun-Connector:Conn_01x01_PTH_1x1mm")
 		(at 106.68 137.16 0)
@@
 			)
 		)
-		(property "Footprint" "SparkFun-Connector:1x01_PTH_1x1mm"
+		(property "Footprint" "SparkFun-Connector:1x01_1x1mm"
 			(at 106.68 144.78 0)
 			(effects
@@
 			)
 		)
-		(property "Footprint" "SparkFun-LED:LED_0402_1005Metric"
+		(property "Footprint" "SparkFun-LED:LED_0402_1005Metric_Red"
 			(at 218.44 71.12 0)
 			(effects
@@
 			)
 		)
-		(property "PROD_ID" "DIO-25000"
+		(property "PROD_ID" "DIO-16757"
 			(at 215.9 71.12 0)
 			(effects

Commit message: Adds axes to design
Parts:
- removed FID1, FID2: Fiducial_0.5mm, SparkFun-Aesthetic:Fiducial_0.5mm_Mask1mm, symbol SparkFun-Aesthetic:Fiducial_0.5mm
Changed lines of the file:
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@@
-	)
-	(symbol
-		(lib_id "SparkFun-Aesthetic:Fiducial_0.5mm")
-		(at 259.08 175.26 0)
-		(unit 1)
-		(exclude_from_sim no)
-		(in_bom yes)
-		(on_board yes)
-		(dnp no)
-		(fields_autoplaced yes)
-		(property "Reference" "FID1"
-			(at 259.08 172.72 0)
-			(effects
-				(font
-					(size 1.27 1.27)
-				)
-				(hide yes)
-			)
-		)
-		(property "Value" "Fiducial_0.5mm"
-			(at 259.08 177.8 0)
-			(effects
-				(font
-					(size 1.27 1.27)
-				)
-				(hide yes)
-			)
-		)
-		(property "Footprint" "SparkFun-Aesthetic:Fiducial_0.5mm_Mask1mm"
-			(at 259.08 180.34 0)
-			(effects
-				(font
-					(size 1.27 1.27)
-				)
-				(hide yes)
-			)
-		)
-		(property "Datasheet" "~"
-			(at 259.08 179.07 0)
-			(effects
-				(font
-					(size 1.27 1.27)
-				)
-				(hide yes)
-			)
-		)
-		(property "Description" "Fiducial Marker"
-			(at 259.08 175.26 0)
-			(effects
-				(font
-					(size 1.27 1.27)
-				)
-				(hide yes)
-			)
-		)
-		(instances
-			(project "SparkFun Indoor Air Quality Sensor - SCD41 SEN55"
-				(path "/e3dd3ae4-244d-4cba-9cca-5d2abf83f29a"
-					(reference "FID1")
-					(unit 1)
-				)
-			)
-		)
 	)
 	(symbol
@@
 		(on_board yes)
 		(dnp no)
-		(fields_autoplaced yes)
 		(property "Reference" "U1"
-			(at 70.866 56.388 0)
-			(effects
-				(font
-					(size 1.27 1.27)
-				)
-				(justify left bottom)
-				(hide yes)
+			(at 72.39 55.118 0)
+			(effects
+				(font
+					(size 1.27 1.27)
+				)
 			)
 		)
 		(property "Value" "LIS3DH"
-			(at 84.836 54.864 0)
-			(effects
-				(font
-					(size 1.27 1.27)
-				)
-				(justify left top)
-				(hide yes)
+			(at 87.884 55.118 0)
+			(effects
+				(font
+					(size 1.27 1.27)
+				)
 			)
 		)
 		(property "Footprint" "SparkFun-Sensor:ST_LGA-16_3x3mm_P0.5mm_5x3"
-			(at 80.518 99.822 0)
+			(at 80.518 93.218 0)
 			(effects
 				(font
@@
 		)
 		(property "Datasheet" "https://www.st.com/en/mems-and-sensors/lis3dh.html"
-			(at 81.28 92.964 0)
+			(at 81.28 86.36 0)
 			(effects
 				(font
@@
 		)
 		(property "Description" "The LIS3DH has dynamically user-selectable full scales of ±2g/±4g/±8g/±16g and is capable of measuring accelerations with output data rates from 1 Hz to 5.3 kHz."
-			(at 82.042 96.266 0)
+			(at 82.042 89.662 0)
 			(effects
 				(font
@@
 		)
 		(property "PROD_ID" "IC-13419"
-			(at 81.534 103.378 0)
+			(at 81.534 96.774 0)
 			(effects
 				(font
@@
 					(unit 1)
 				)
-			)
-		)
-	)
-	(symbol
-		(lib_id "SparkFun-Aesthetic:Fiducial_0.5mm")
-		(at 259.08 179.07 0)
-		(unit 1)
-		(exclude_from_sim no)
-		(in_bom yes)
-		(on_board yes)
-		(dnp no)
-		(fields_autoplaced yes)
-		(property "Reference" "FID2"
-			(at 259.08 176.53 0)
-			(effects
-				(font
-					(size 1.27 1.27)
-				)
-				(hide yes)
-			)
-		)
-		(property "Value" "Fiducial_0.5mm"
-			(at 259.08 181.61 0)
-			(effects
-				(font
-					(size 1.27 1.27)
-				)
-				(hide yes)
-			)
-		)
-		(property "Footprint" "SparkFun-Aesthetic:Fiducial_0.5mm_Mask1mm"
-			(at 259.08 184.15 0)
-			(effects
-				(font
-					(size 1.27 1.27)
-				)
-				(hide yes)
-			)
-		)
-		(property "Datasheet" "~"
-			(at 259.08 182.88 0)
-			(effects
-				(font
-					(size 1.27 1.27)
-				)
-				(hide yes)
-			)
-		)
-		(property "Description" "Fiducial Marker"
-			(at 259.08 179.07 0)
-			(effects
-				(font
-					(size 1.27 1.27)
-				)
-				(hide yes)
-			)
-		)
-		(instances
-			(project "SparkFun Indoor Air Quality Sensor - SCD41 SEN55"
-				(path "/e3dd3ae4-244d-4cba-9cca-5d2abf83f29a"
-					(reference "FID2")
-					(unit 1)
-				)
